File: eagle_main/arduino_shield/shield_schematic.brd (EAGLE design)
At the start: 100 x 80 mm, 17 parts, among them IC1 74LS595D, J1 ARDUINO_R3_SHIELD

Commit message: Updated parts for November 4th
Parts:
- removed C1: 0.1uF, SparkFun-Capacitors:0603-CAP
- removed D1, D10, D2, D3, D4, D5, D6, D7, D8, D9: (no value), SparkFun-LED:LED5MM
- removed IC1: 74LS595D, SparkFun-DigitalIC:SO16
- removed R1: (no value), SparkFun-Resistors:0603-RES
- added LED1, LED2, LED3, LED4, LED5, LED6: APA102SMD, Arduino_Shield:RGBLED5050
- moved U$1 38.6 mm to (43.9, 59.9), turned to 180 degrees
- moved SG1 17.8 mm to (19.1, 63.5), turned to 180 degrees
Connections:
- removed net N$4: IC1.11, J1.D4
- removed net N$5: IC1.12, J1.D5
- removed net N$6: IC1.10, R1.1
- removed net N$8: IC1.14, J1.D6
- new net LED_CI: J1.D13, LED1.CI
- new net LED_DI: J1.D11, LED1.DI
- new net N$14: LED1.DO, LED2.DI
- new net N$15: LED1.CO, LED2.CI
- new net N$16: LED2.DO, LED3.DI
- new net N$17: LED2.CO, LED3.CI
- new net N$18: LED3.CO, LED4.CI
- new net N$19: LED3.DO, LED4.DI
- new net N$20: LED4.CO, LED5.CI
- new net N$21: LED4.DO, LED5.DI
- new net N$22: LED5.DO, LED6.DI
- new net N$23: LED5.CO, LED6.CI
- net GND: now also LED1.GND, LED2.GND, LED3.GND, LED4.GND, LED5.GND, LED6.GND; no longer C1.2, IC1.13, IC1.8
- net VIN: now also LED1.VCC, LED2.VCC, LED3.VCC, LED4.VCC, LED5.VCC, LED6.VCC; no longer C1.1, IC1.16, R1.2
Routing:
- net N$1: track 47.4 -> 8.77 mm
- net N$8: track 21.5 -> 0.00 mm
- net N$5: track 21.2 -> 0.00 mm
- net N$4: track 20.7 -> 0.00 mm
- net GND: track 25.9 -> 5.59 mm, vias 4 -> 1
- net LED_DI: track 0.00 -> 19.9 mm
- net VIN: track 75.4 -> 94.3 mm
- net N$3: track 28.2 -> 9.45 mm
- net LED_CI: track 0.00 -> 16.9 mm
- net N$6: track 9.10 -> 0.00 mm
- net N$21: track 0.00 -> 4.98 mm
- net N$20: track 0.00 -> 4.98 mm
- net N$17: track 0.00 -> 4.73 mm
- net N$16: track 0.00 -> 4.73 mm
- net N$15: track 0.00 -> 4.73 mm
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Other:
- board text added: "Learning Committee Shield Created by John Lee 11/4/2015"
